Commit message: Added basic urdf file and updated launch and CMake files to accomodate rviz

File: src/hexapod_nodes/urdf/hexapod.urdf.xacro (robot description, xacro)
@@ -0,0 +1,15 @@
+<?xml version="1.0"?>
+<robot xmlns:xacro="http://www.ros.org/wiki/xacro" name="hexapod">
+<xacro:property name="segment_1_radius" value="0.2"/>
+<xacro:property name="segment_1_length" value="1"/>
+<xacro:macro name="leg" params="leg_id">
+    <link name="leg+${leg_id}_segment_1">
+        <visual>
+            <geometry>
+                <cylinder length="${segment_1_length}" radius="${segment_1_radius}"/>
+            </geometry>
+        </visual>
+    </link>
+</xacro:macro>
+<xacro:leg leg_id="1"/>
+</robot>

Commit message: Fixed some issues with the URDF

File: src/hexapod_nodes/urdf/hexapod.urdf.xacro (robot description, xacro)
@@ -1,15 +1,56 @@
 <?xml version="1.0"?>
 <robot xmlns:xacro="http://www.ros.org/wiki/xacro" name="hexapod">
-<xacro:property name="segment_1_radius" value="0.2"/>
-<xacro:property name="segment_1_length" value="1"/>
-<xacro:macro name="leg" params="leg_id">
-    <link name="leg+${leg_id}_segment_1">
+    <xacro:property name="body_radius" value="1"/>
+    <xacro:property name="segment_1_radius" value="0.2"/>
+    <xacro:property name="segment_1_length" value="1"/>
+    <material name="white">
+        <color rgba="1 1 1 1"/>
+    </material>
+    <xacro:macro name="default_inertial" params="mass">
+        <inertial>
+            <mass value="${mass}"/>
+            <inertia ixx="1e-3" ixy="0.0" ixz="0.0" iyy="1e-3" iyz="0.0" izz="1e-3"/>
+        </inertial>
+    </xacro:macro>
+    <link name="body">
         <visual>
             <geometry>
-                <cylinder length="${segment_1_length}" radius="${segment_1_radius}"/>
+                <sphere radius="${body_radius}"/>
             </geometry>
+            <material name="white"/>
         </visual>
+        <collision>
+            <geometry>
+                <sphere radius="${body_radius}"/>
+            </geometry>
+        </collision>
+        <!--
+        <xacro:default_inertial mass="10"/>
+        -->
     </link>
-</xacro:macro>
-<xacro:leg leg_id="1"/>
+    <xacro:macro name="leg" params="leg_id">
+        <link name="leg_${leg_id}_segment_1">
+            <visual>
+                <geometry>
+                    <cylinder length="${segment_1_length}" radius="${segment_1_radius}"/>
+                </geometry>
+                <material name="white"/>
+            </visual>
+            <collision>
+                <geometry>
+                    <cylinder length="${segment_1_length}" radius="${segment_1_radius}"/>
+                </geometry>
+                <origin xyz = "0 0 -${segment_1_length/2}" rpy="0 ${pi/2} 0"/>
+            </collision>
+            <xacro:default_inertial mass="10"/>
+        </link>
+        <joint name="$body_segment_1_joint" type="revolute">
+            <axis xzy="0 0 1"/>
+            <limit effort="1000.0" lower="0.0" upper="0.548" velocity="0.5"/>
+            <parent link="body"/>
+            <child link="leg_${leg_id}_segment_1"/>
+            <origin xyz="0 0 0"/>
+        </joint>
+    </xacro:macro>
+    <xacro:leg leg_id="1"/>
 </robot>

Commit message: Some minor changes to the URDF

File: src/hexapod_nodes/urdf/hexapod.urdf.xacro (robot description, xacro)
@@ -50,5 +50,5 @@
             <parent link="body"/>
             <child link="leg_${leg_id}_segment_1"/>
-            <origin xyz="0 0 0"/>
+            <origin xyz="${body_radius} 0 0"/>
         </joint>
     </xacro:macro>

Commit message: Removed gui parameter from launch file since it was causing problems. There is now no way to launch rviz without joint_state_publisher_gui.

File: src/hexapod_nodes/urdf/hexapod.urdf.xacro (robot description, xacro)
@@ -3,5 +3,5 @@
     <xacro:property name="body_radius" value="1"/>
     <xacro:property name="segment_1_radius" value="0.2"/>
-    <xacro:property name="segment_1_length" value="1"/>
+    <xacro:property name="segment_1_length" value="3"/>
     <material name="white">
         <color rgba="1 1 1 1"/>
@@ -41,9 +41,9 @@
                     <cylinder length="${segment_1_length}" radius="${segment_1_radius}"/>
                 </geometry>
-                <origin xyz = "0 0 -${segment_1_length/2}" rpy="0 ${pi/2} 0"/>
+                <origin xyz = "0 0 -${segment_1_length/2}" rpy="0 1.5705 0"/>
             </collision>
             <xacro:default_inertial mass="10"/>
         </link>
-        <joint name="$body_segment_1_joint" type="revolute">
+        <joint name="$leg_${leg_id}_joint_1" type="revolute">
             <axis xzy="0 0 1"/>
             <limit effort="1000.0" lower="0.0" upper="0.548" velocity="0.5"/>

Commit message: Made basic URDF model with all fixed joints.

File: src/hexapod_nodes/urdf/hexapod.urdf.xacro (robot description, xacro)
@@ -1,7 +1,9 @@
 <?xml version="1.0"?>
 <robot xmlns:xacro="http://www.ros.org/wiki/xacro" name="hexapod">
-    <xacro:property name="body_radius" value="1"/>
-    <xacro:property name="segment_1_radius" value="0.2"/>
-    <xacro:property name="segment_1_length" value="3"/>
+    <xacro:property name="body_radius" value="0.5"/>
+    <xacro:property name="leg_radius" value="0.2"/>
+    <xacro:property name="segment_0_length" value="0.5"/>
+    <xacro:property name="segment_1_length" value="1"/>
+    <xacro:property name="segment_2_length" value="2"/>
     <material name="white">
         <color rgba="1 1 1 1"/>
@@ -29,28 +31,88 @@
         -->
     </link>
+    <!-- Definition of an individual leg of the robot -->
     <xacro:macro name="leg" params="leg_id">
-        <link name="leg_${leg_id}_segment_1">
+        <!-- First segment -->
+        <link name="leg_${leg_id}_segment_0">
             <visual>
                 <geometry>
-                    <cylinder length="${segment_1_length}" radius="${segment_1_radius}"/>
+                    <cylinder length="${segment_0_length}" radius="${leg_radius}"/>
                 </geometry>
+                <origin xyz="0 0 ${segment_0_length/2}"/>
                 <material name="white"/>
             </visual>
             <collision>
                 <geometry>
-                    <cylinder length="${segment_1_length}" radius="${segment_1_radius}"/>
+                    <cylinder length="${segment_0_length}" radius="${leg_radius}"/>
                 </geometry>
-                <origin xyz = "0 0 -${segment_1_length/2}" rpy="0 1.5705 0"/>
+                <origin xyz="0 0 ${segment_0_length/2}"/>
             </collision>
             <xacro:default_inertial mass="10"/>
         </link>
-        <joint name="$leg_${leg_id}_joint_1" type="revolute">
-            <axis xzy="0 0 1"/>
-            <limit effort="1000.0" lower="0.0" upper="0.548" velocity="0.5"/>
+        <!-- Joint connecting body to leg -->
+        <joint name="$leg_${leg_id}_joint_0" type="fixed">
+            <!-- <axis xzy="0 0 1"/> -->
+            <!-- <limit effort="1000.0" lower="0.0" upper="0.548" velocity="0.5"/> -->
             <parent link="body"/>
+            <child link="leg_${leg_id}_segment_0"/>
+            <!-- Places legs with the correct position and rotation based on their ID -->
+            <origin xyz="${body_radius*sin(leg_id*pi/3)} ${body_radius*cos(leg_id*pi/3)} 0" rpy="0 ${pi/2} ${pi/2-leg_id*pi/3}"/>
+        </joint>
+        <!-- Second segment -->
+        <link name="leg_${leg_id}_segment_1">
+            <visual>
+                <geometry>
+                    <cylinder length="${segment_1_length}" radius="${leg_radius}"/>
+                </geometry>
+                <origin xyz="0 0 ${segment_1_length/2}"/>
+                <material name="white"/>
+            </visual>
+            <collision>
+                <geometry>
+                    <cylinder length="${segment_1_length}" radius="${leg_radius}"/>
+                </geometry>
+                <origin xyz="0 0 ${segment_1_length/2}"/>
+            </collision>
+            <xacro:default_inertial mass="10"/>
+        </link>
+        <!-- Joint connecting first and second segments -->
+        <joint name="$leg_${leg_id}_joint_1" type="fixed">
+            <!-- <axis xzy="0 0 1"/> -->
+            <!-- <limit effort="1000.0" lower="0.0" upper="0.548" velocity="0.5"/> -->
+            <parent link="leg_${leg_id}_segment_0"/>
             <child link="leg_${leg_id}_segment_1"/>
-            <origin xyz="${body_radius} 0 0"/>
+            <origin xyz="0 0 ${segment_0_length}" rpy="0 0 0"/>
+        </joint>
+        <!-- Third segment -->
+        <link name="leg_${leg_id}_segment_2">
+            <visual>
+                <geometry>
+                    <cylinder length="${segment_2_length}" radius="${leg_radius}"/>
+                </geometry>
+                <origin xyz="0 0 ${segment_2_length/2}"/>
+                <material name="white"/>
+            </visual>
+            <collision>
+                <geometry>
+                    <cylinder length="${segment_2_length}" radius="${leg_radius}"/>
+                </geometry>
+                <origin xyz="0 0 ${segment_2_length/2}"/>
+            </collision>
+            <xacro:default_inertial mass="10"/>
+        </link>
+        <!-- Joint connecting second and third segments -->
+        <joint name="$leg_${leg_id}_joint_2" type="fixed">
+            <!-- <axis xzy="0 0 1"/> -->
+            <!-- <limit effort="1000.0" lower="0.0" upper="0.548" velocity="0.5"/> -->
+            <parent link="leg_${leg_id}_segment_1"/>
+            <child link="leg_${leg_id}_segment_2"/>
+            <origin xyz="0 0 ${segment_1_length}" rpy="0 0 0"/>
         </joint>
     </xacro:macro>
+    <xacro:leg leg_id="0"/>
     <xacro:leg leg_id="1"/>
+    <xacro:leg leg_id="2"/>
+    <xacro:leg leg_id="3"/>
+    <xacro:leg leg_id="4"/>
+    <xacro:leg leg_id="5"/>
 </robot>

Commit message: I have no idea what I did but I fixed the URDF issue

File: src/hexapod_nodes/urdf/hexapod.urdf.xacro (robot description, xacro)
@@ -1,4 +1,5 @@
 <?xml version="1.0"?>
 <robot xmlns:xacro="http://www.ros.org/wiki/xacro" name="hexapod">
+    <!-- Constants used throughout the model -->
     <xacro:property name="body_radius" value="0.5"/>
     <xacro:property name="leg_radius" value="0.2"/>
@@ -6,13 +7,18 @@
     <xacro:property name="segment_1_length" value="1"/>
     <xacro:property name="segment_2_length" value="2"/>
+    <!-- Some colors used throughout the model -->
     <material name="white">
         <color rgba="1 1 1 1"/>
     </material>
-    <xacro:macro name="default_inertial" params="mass">
-        <inertial>
-            <mass value="${mass}"/>
-            <inertia ixx="1e-3" ixy="0.0" ixz="0.0" iyy="1e-3" iyz="0.0" izz="1e-3"/>
-        </inertial>
-    </xacro:macro>
+    <material name="red">
+        <color rgba="1 0 0 1"/>
+    </material>
+    <material name="green">
+        <color rgba="0 1 0 1"/>
+    </material>
+    <material name="blue">
+        <color rgba="0 0 1 1"/>
+    </material>
+    <!-- The main body of the robot -->
     <link name="body">
         <visual>
@@ -27,11 +33,8 @@
             </geometry>
         </collision>
-        <!--
-        <xacro:default_inertial mass="10"/>
-        -->
     </link>
-    <!-- Definition of an individual leg of the robot -->
+    <!-- Macro used to generate legs -->
     <xacro:macro name="leg" params="leg_id">
-        <!-- First segment -->
+        <!-- First leg segment -->
         <link name="leg_${leg_id}_segment_0">
             <visual>
@@ -39,6 +42,6 @@
                     <cylinder length="${segment_0_length}" radius="${leg_radius}"/>
                 </geometry>
+                <material name="blue"/>
                 <origin xyz="0 0 ${segment_0_length/2}"/>
-                <material name="white"/>
             </visual>
             <collision>
@@ -48,16 +51,15 @@
                 <origin xyz="0 0 ${segment_0_length/2}"/>
             </collision>
-            <xacro:default_inertial mass="10"/>
         </link>
-        <!-- Joint connecting body to leg -->
-        <joint name="$leg_${leg_id}_joint_0" type="fixed">
-            <!-- <axis xzy="0 0 1"/> -->
-            <!-- <limit effort="1000.0" lower="0.0" upper="0.548" velocity="0.5"/> -->
+        <!-- Joint connecting body to first leg segment -->
+        <joint name="body_to_leg_${leg_id}_segment_0" type="revolute">
             <parent link="body"/>
             <child link="leg_${leg_id}_segment_0"/>
-            <!-- Places legs with the correct position and rotation based on their ID -->
+            <axis xyz="1 0 0"/>
+            <limit effort="1000.0" lower="-0.5" upper="0.5" velocity="0.5"/>
+            <!-- Determines the position and orientation of the leg based on its ID -->
             <origin xyz="${body_radius*sin(leg_id*pi/3)} ${body_radius*cos(leg_id*pi/3)} 0" rpy="0 ${pi/2} ${pi/2-leg_id*pi/3}"/>
         </joint>
-        <!-- Second segment -->
+        <!-- Second leg segment -->
         <link name="leg_${leg_id}_segment_1">
             <visual>
@@ -65,6 +67,6 @@
                     <cylinder length="${segment_1_length}" radius="${leg_radius}"/>
                 </geometry>
+                <material name="red"/>
                 <origin xyz="0 0 ${segment_1_length/2}"/>
-                <material name="white"/>
             </visual>
             <collision>
@@ -74,15 +76,14 @@
                 <origin xyz="0 0 ${segment_1_length/2}"/>
             </collision>
-            <xacro:default_inertial mass="10"/>
         </link>
-        <!-- Joint connecting first and second segments -->
-        <joint name="$leg_${leg_id}_joint_1" type="fixed">
-            <!-- <axis xzy="0 0 1"/> -->
-            <!-- <limit effort="1000.0" lower="0.0" upper="0.548" velocity="0.5"/> -->
+        <!-- Joint connecting first and second leg segments -->
+        <joint name="leg_${leg_id}_segment_0_to_segment_1" type="revolute">
+            <axis xyz="0 1 0"/>
             <parent link="leg_${leg_id}_segment_0"/>
             <child link="leg_${leg_id}_segment_1"/>
-            <origin xyz="0 0 ${segment_0_length}" rpy="0 0 0"/>
+            <limit effort="1000.0" lower="-0.5" upper="0.5" velocity="0.5"/>
+            <origin xyz="0 0 ${segment_1_length}"/>
         </joint>
-        <!-- Third segment -->
+        <!-- Third leg segment -->
         <link name="leg_${leg_id}_segment_2">
             <visual>
@@ -90,6 +91,6 @@
                     <cylinder length="${segment_2_length}" radius="${leg_radius}"/>
                 </geometry>
+                <material name="green"/>
                 <origin xyz="0 0 ${segment_2_length/2}"/>
-                <material name="white"/>
             </visual>
             <collision>
@@ -99,13 +100,12 @@
                 <origin xyz="0 0 ${segment_2_length/2}"/>
             </collision>
-            <xacro:default_inertial mass="10"/>
         </link>
-        <!-- Joint connecting second and third segments -->
-        <joint name="$leg_${leg_id}_joint_2" type="fixed">
-            <!-- <axis xzy="0 0 1"/> -->
-            <!-- <limit effort="1000.0" lower="0.0" upper="0.548" velocity="0.5"/> -->
+        <!-- Joint connecting second and third leg segments -->
+        <joint name="leg_${leg_id}_segment_1_to_segment_2" type="revolute">
+            <axis xyz="0 1 0"/>
             <parent link="leg_${leg_id}_segment_1"/>
             <child link="leg_${leg_id}_segment_2"/>
-            <origin xyz="0 0 ${segment_1_length}" rpy="0 0 0"/>
+            <limit effort="1000.0" lower="-0.5" upper="0.5" velocity="0.5"/>
+            <origin xyz="0 0 ${segment_2_length}"/>
         </joint>
     </xacro:macro>

Commit message: small fix to the URDF file

File: src/hexapod_nodes/urdf/hexapod.urdf.xacro (robot description, xacro)
@@ -83,5 +83,5 @@
             <child link="leg_${leg_id}_segment_1"/>
             <limit effort="1000.0" lower="-0.5" upper="0.5" velocity="0.5"/>
-            <origin xyz="0 0 ${segment_1_length}"/>
+            <origin xyz="0 0 ${segment_1_length/2}"/>
         </joint>
         <!-- Third leg segment -->
@@ -107,5 +107,5 @@
             <child link="leg_${leg_id}_segment_2"/>
             <limit effort="1000.0" lower="-0.5" upper="0.5" velocity="0.5"/>
-            <origin xyz="0 0 ${segment_2_length}"/>
+            <origin xyz="0 0 ${segment_2_length/2}"/>
         </joint>
     </xacro:macro>

Commit message: Started implementing tf2 broadcaster

File: src/hexapod_nodes/urdf/hexapod.urdf.xacro (robot description, xacro)
@@ -82,5 +82,5 @@
             <parent link="leg_${leg_id}_segment_0"/>
             <child link="leg_${leg_id}_segment_1"/>
-            <limit effort="1000.0" lower="-0.5" upper="0.5" velocity="0.5"/>
+            <limit effort="1000.0" lower="-${2*pi/3}" upper="${2*pi/3}" velocity="0.5"/>
             <origin xyz="0 0 ${segment_1_length/2}"/>
         </joint>
@@ -106,5 +106,5 @@
             <parent link="leg_${leg_id}_segment_1"/>
             <child link="leg_${leg_id}_segment_2"/>
-            <limit effort="1000.0" lower="-0.5" upper="0.5" velocity="0.5"/>
+            <limit effort="1000.0" lower="-${2*pi/3}" upper="${2*pi/3}" velocity="0.5"/>
             <origin xyz="0 0 ${segment_2_length/2}"/>
         </joint>

Commit message: Reworked leg_state_broadcaster to use the robot definition from the URDF file and to send joint_state messages to the robot_state_publisher rather than directly sending tf2 messages.

File: src/hexapod_nodes/urdf/hexapod.urdf.xacro (robot description, xacro)
@@ -53,5 +53,5 @@
         </link>
         <!-- Joint connecting body to first leg segment -->
-        <joint name="body_to_leg_${leg_id}_segment_0" type="revolute">
+        <joint name="leg_${leg_id}_body_to_segment_0" type="revolute">
             <parent link="body"/>
             <child link="leg_${leg_id}_segment_0"/>

Commit message: Reworked leg state format to be a simpler cartesian coordinate system centered on the base joint of the leg. Updated inverse kinematics accordingly.

File: src/hexapod_nodes/urdf/hexapod.urdf.xacro (robot description, xacro)
@@ -5,5 +5,5 @@
     <xacro:property name="leg_radius" value="0.2"/>
     <xacro:property name="segment_0_length" value="0.5"/>
-    <xacro:property name="segment_1_length" value="1"/>
+    <xacro:property name="segment_1_length" value="2"/>
     <xacro:property name="segment_2_length" value="2"/>
     <!-- Some colors used throughout the model -->
@@ -83,5 +83,5 @@
             <child link="leg_${leg_id}_segment_1"/>
             <limit effort="1000.0" lower="-${2*pi/3}" upper="${2*pi/3}" velocity="0.5"/>
-            <origin xyz="0 0 ${segment_1_length/2}"/>
+            <origin xyz="0 0 ${segment_0_length}"/>
         </joint>
         <!-- Third leg segment -->
@@ -107,5 +107,5 @@
             <child link="leg_${leg_id}_segment_2"/>
             <limit effort="1000.0" lower="-${2*pi/3}" upper="${2*pi/3}" velocity="0.5"/>
-            <origin xyz="0 0 ${segment_2_length/2}"/>
+            <origin xyz="0 0 ${segment_1_length}"/>
         </joint>
     </xacro:macro>
